File: KiCAD/BT-Modul.kicad_pcb (KiCad board)
At the start: 2 copper layers, 63.5 x 63.5 mm, 17 parts, among them P1 CONN_01X03, P2 USB_B, P3 USB_A, U1 KRC-86B, U2 ICL7660S, U3 opa2134

Commit message: Ready for ordering
Other:
- board text added: "https://github.com/tht/BT-Module"
Changed lines of the file:
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@@
   (general
     (links 34)
-    (no_connects 1)
+    (no_connects 0)
     (area 60 60 130.000001 130.000001)
     (thickness 1.6)
-    (drawings 18)
+    (drawings 19)
     (tracks 180)
     (zones 0)
@@
     (visible_elements FFFFFF7F)
     (pcbplotparams
-      (layerselection 0x00030_80000001)
-      (usegerberextensions false)
+      (layerselection 0x010f0_80000001)
+      (usegerberextensions true)
       (excludeedgelayer true)
       (linewidth 0.100000)
@@
       (outputformat 1)
       (mirror false)
-      (drillshape 1)
+      (drillshape 0)
       (scaleselection 1)
-      (outputdirectory ""))
+      (outputdirectory gerber))
   )
   (net 0 "")
@@
       (net 2 GND))
   )
+  (gr_text https://github.com/tht/BT-Module (at 95 79.125) (layer B.SilkS)
+    (effects (font (size 1.5 1.5) (thickness 0.3)) (justify mirror))
+  )
   (gr_text "31.62mm\n28.28mm" (at 90 70) (layer B.SilkS)

Commit message: Rev 1 as ordered
Other:
- board text added: "rev 1 2017/03"
- board text removed: "rev 1 2017/02"
Changed lines of the file:
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@@
   (module BTA:USB_A_Fem_Vert (layer F.Cu)
     (at 69.6 95 270)
-    (fp_text reference P3 (at 0 3.81 270) (layer F.SilkS)
+    (fp_text reference P3 (at 0 3.81 270) (layer F.SilkS) hide
       (effects (font (size 1 1) (thickness 0.15)))
     )
@@
     (effects (font (size 1.5 1.5) (thickness 0.3)))
   )
-  (gr_text "rev 1  2017/02" (at 95 123.575) (layer F.SilkS)
+  (gr_text "rev 1  2017/03" (at 95 123.575) (layer F.SilkS)
     (effects (font (size 1.5 1.5) (thickness 0.3)))
   )
